File: Schematic/AGC_Disabler/AGC_Disabler.kicad_pcb (KiCad board)
At the start: 2 copper layers, 46 x 22.5 mm, 19 parts, among them J1 Batt+, J2 Out+, J3 Batt-, J4 Out-, SW1 SW_DPDT_x2, SW2 SW_DPDT_x2, U1 TLV76601, U2 LED_Voltmeter_0.28

Commit message: File cleanup
Parts:
- removed R1, R3: 0Ω, Resistor_SMD:R_0603_1608Metric_Pad0.98x0.95mm_HandSolder
- moved RV1 4.99 mm to (114.5, 65.3), turned to -90 degrees
Connections:
- RV1 pad 2: Net-(R1-Pad2) -> Net-(U1-FB)
Routing:
- net Net-(R1-Pad2): track 15.2 -> 0.00 mm
- net Net-(SW1B-B): track 40.8 -> 48.1 mm
- net Net-(U1-FB): track 13.9 -> 20.2 mm
Other:
- board text added: "AGC Disabler R0164C_2412_Pb Bjørner Sandom"
- board text removed: "AGC Disabler R0164B_2410 Bjørner Sandom"
