File: Schematic/AGC_Disabler/AGC_Disabler.kicad_sch (KiCad schematic)
At the start: 18 parts, among them J1 Batt+, J2 Out+, J3 Batt-, J4 Out-, SW1 SW_DPDT_x2, SW2 SW_DPDT_x2, U1 TLV76601, U2 LED_Voltmeter_0.28

Commit message: File cleanup
Parts:
- removed R1, R3: 0Ω, Resistor_SMD:R_0603_1608Metric_Pad0.98x0.95mm_HandSolder, symbol Device:R_Small
Connections:
- net at RV1.2: now also R4.1, RV1.3, U1.3 (FB)
Other:
- note added: "Vout=0.8*(1+RV1/R4)"
- note removed: "Vout=0.8*(1+RV1/R1)"
Changed lines of the file:
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@@
   (junction (at 128.905 85.725) (diameter 0) (color 0 0 0 0)
   )
-  (junction (at 154.94 71.12) (diameter 0) (color 0 0 0 0)
-  )
   (junction (at 121.92 66.675) (diameter 0) (color 0 0 0 0)
   )
   (junction (at 95.885 66.675) (diameter 0) (color 0 0 0 0)
   )
-  (junction (at 146.685 66.675) (diameter 0) (color 0 0 0 0)
-  )
   (junction (at 160.02 85.725) (diameter 0) (color 0 0 0 0)
   )
@@
   (junction (at 116.205 66.675) (diameter 0) (color 0 0 0 0)
   )
+  (junction (at 150.495 74.295) (diameter 0) (color 0 0 0 0)
+  )
   (junction (at 160.02 76.835) (diameter 0) (color 0 0 0 0)
   )
   (junction (at 131.445 85.725) (diameter 0) (color 0 0 0 0)
-  )
-  (junction (at 146.685 74.295) (diameter 0) (color 0 0 0 0)
   )
   (junction (at 171.45 85.725) (diameter 0) (color 0 0 0 0)
@@
     (stroke (width 0) (type default))
   )
-  (wire (pts (xy 154.94 71.12) (xy 157.48 71.12))
-    (stroke (width 0) (type default))
-  )
   (wire (pts (xy 118.745 119.38) (xy 118.745 123.825))
     (stroke (width 0) (type default))
@@
     (stroke (width 0) (type default))
   )
+  (wire (pts (xy 139.065 74.295) (xy 150.495 74.295))
+    (stroke (width 0) (type default))
+  )
   (wire (pts (xy 171.45 78.105) (xy 171.45 85.725))
     (stroke (width 0) (type default))
   )
-  (wire (pts (xy 139.065 74.295) (xy 146.685 74.295))
-    (stroke (width 0) (type default))
-  )
   (wire (pts (xy 116.205 85.725) (xy 128.905 85.725))
     (stroke (width 0) (type default))
@@
     (stroke (width 0) (type default))
   )
-  (wire (pts (xy 146.685 74.295) (xy 146.685 76.835))
+  (wire (pts (xy 150.495 74.295) (xy 150.495 76.835))
     (stroke (width 0) (type default))
   )
@@
     (stroke (width 0) (type default))
   )
-  (wire (pts (xy 148.59 69.85) (xy 146.685 69.85))
-    (stroke (width 0) (type default))
-  )
   (wire (pts (xy 131.445 85.725) (xy 160.02 85.725))
     (stroke (width 0) (type default))
@@
     (stroke (width 0) (type default))
   )
-  (wire (pts (xy 146.685 66.675) (xy 160.02 66.675))
-    (stroke (width 0) (type default))
-  )
   (wire (pts (xy 105.41 66.675) (xy 116.205 66.675))
     (stroke (width 0) (type default))
@@
     (stroke (width 0) (type default))
   )
-  (wire (pts (xy 148.59 72.39) (xy 146.685 72.39))
-    (stroke (width 0) (type default))
-  )
-  (wire (pts (xy 139.065 66.675) (xy 146.685 66.675))
+  (wire (pts (xy 139.065 66.675) (xy 160.02 66.675))
     (stroke (width 0) (type default))
   )
@@
     (stroke (width 0) (type default))
   )
-  (wire (pts (xy 146.685 72.39) (xy 146.685 74.295))
-    (stroke (width 0) (type default))
-  )
-  (wire (pts (xy 154.94 71.12) (xy 154.94 72.39))
+  (wire (pts (xy 150.495 71.12) (xy 150.495 74.295))
     (stroke (width 0) (type default))
   )
@@
     (stroke (width 0) (type default))
   )
-  (wire (pts (xy 153.67 69.85) (xy 154.94 69.85))
-    (stroke (width 0) (type default))
-  )
   (wire (pts (xy 160.02 85.725) (xy 171.45 85.725))
     (stroke (width 0) (type default))
@@
     (stroke (width 0) (type default))
   )
-  (wire (pts (xy 153.67 72.39) (xy 154.94 72.39))
+  (wire (pts (xy 150.495 71.12) (xy 157.48 71.12))
     (stroke (width 0) (type default))
   )
@@
     (stroke (width 0) (type default))
   )
-  (wire (pts (xy 154.94 69.85) (xy 154.94 71.12))
-    (stroke (width 0) (type default))
-  )
   (wire (pts (xy 128.905 85.725) (xy 131.445 85.725))
     (stroke (width 0) (type default))
@@
     (stroke (width 0) (type default))
   )
-  (wire (pts (xy 146.685 76.835) (xy 160.02 76.835))
+  (wire (pts (xy 150.495 76.835) (xy 160.02 76.835))
     (stroke (width 0) (type default))
   )
@@
     (stroke (width 0) (type default))
   )
-  (wire (pts (xy 146.685 69.85) (xy 146.685 66.675))
-    (stroke (width 0) (type default))
-  )
   (wire (pts (xy 117.475 131.445) (xy 117.475 130.81))
     (stroke (width 0) (type default))
   )
-  (text "Vout=0.8*(1+RV1/R1)" (at 142.875 88.9 0)
+  (text "Vout=0.8*(1+RV1/R4)" (at 142.875 88.9 0)
     (effects (font (size 1.27 1.27)) (justify left bottom))
   )
@@
         (path "/bc1c57a6-6d64-4e0c-b91d-cea1dd9bb183"
           (reference "D2") (unit 1)
-        )
-      )
-    )
-  )
-  (symbol (lib_id "Device:R_Small") (at 151.13 72.39 90) (mirror x) (unit 1)
-    (in_bom yes) (on_board yes) (dnp no)
-    (property "Reference" "R3" (at 150.495 74.295 90)
-      (effects (font (size 1.27 1.27)) (justify left))
-    )
-    (property "Value" "0Ω" (at 154.305 74.295 90)
-      (effects (font (size 1.27 1.27)) (justify left))
-    )
-    (property "Footprint" "Resistor_SMD:R_0603_1608Metric_Pad0.98x0.95mm_HandSolder" (at 151.13 72.39 0)
-      (effects (font (size 1.27 1.27)) hide)
-    )
-    (property "Datasheet" "~" (at 151.13 72.39 0)
-      (effects (font (size 1.27 1.27)) hide)
-    )
-    (property "Comments" "" (at 151.13 72.39 0)
-      (effects (font (size 1.27 1.27)))
-    )
-    (pin "1")
-    (pin "2")
-    (instances
-      (project "AGC_Disabler"
-        (path "/bc1c57a6-6d64-4e0c-b91d-cea1dd9bb183"
-          (reference "R3") (unit 1)
         )
       )
@@
         )
       )
-    )
-  )
-  (symbol (lib_id "Device:R_Small") (at 151.13 69.85 90) (unit 1)
-    (in_bom yes) (on_board yes) (dnp yes)
-    (property "Reference" "R1" (at 150.495 67.945 90)
-      (effects (font (size 1.27 1.27)) (justify left))
-    )
-    (property "Value" "0Ω" (at 154.305 67.945 90)
-      (effects (font (size 1.27 1.27)) (justify left))
-    )
-    (property "Footprint" "Resistor_SMD:R_0603_1608Metric_Pad0.98x0.95mm_HandSolder" (at 151.13 69.85 0)
-      (effects (font (size 1.27 1.27)) hide)
-    )
-    (property "Datasheet" "~" (at 151.13 69.85 0)
-      (effects (font (size 1.27 1.27)) hide)
-    )
-    (property "Comments" "" (at 151.13 69.85 0)
-      (effects (font (size 1.27 1.27)))
-    )
-    (pin "1")
-    (pin "2")
-    (instances
-      (project "AGC_Disabler"
-        (path "/bc1c57a6-6d64-4e0c-b91d-cea1dd9bb183"
-          (reference "R1") (unit 1)
-        )
-      )
